File: board/proto1/proto1.kicad_pcb (KiCad board)
At the start: 2 copper layers, 88 parts, among them J1 Micro_SD_Card_Det, J10 GND, J11 J11, J11A1 J11A, J12 VBatt, J13 VBattSw, J14 LCD, J15 3.3V Out, J2 LED_DOUT, J3 Expansion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

Commit message: more layout work
Parts:
- C10, C11, C12, C13, C14, C15, C16, C17, C18, C3, C4, C5, C6, C7, C8, C9, J14, R8: moved to B.Cu
- moved SW1 184.1 mm to (92.0, 151.0)
- moved R3 180.0 mm to (106.2, 154.8)
- moved C28 175.7 mm to (106.2, 167.0)
- moved C2 164.2 mm to (98.8, 116.5)
- moved R4 163.2 mm to (106.2, 159.5)
- moved C25 153.0 mm to (106.2, 151.8), turned to 180 degrees
- moved C3 147.3 mm to (118.2, 30.5), turned to 270 degrees
- moved C26 143.8 mm to (106.2, 157.2)
- moved C29 141.2 mm to (158.0, 164.0)
- moved C7 140.7 mm to (118.2, 37.5), turned to 270 degrees
- moved SW2 140.6 mm to (88.0, 156.2)
- moved C4 139.1 mm to (126.5, 30.5), turned to 270 degrees
- moved C27 138.6 mm to (106.2, 162.2)
- moved R2 136.8 mm to (106.2, 149.0)
- moved C12 134.3 mm to (126.5, 44.5), turned to 270 degrees
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Other:
- board outline added: 77.5 x 101.8 mm

Commit message: lots more layout work
Parts:
- removed C23, C24: 0.1, Capacitors_SMD:C_0805
- C21, C22: moved to B.Cu
- moved C22 52.3 mm to (143.0, 51.6), turned to 90 degrees
- moved J2 48.3 mm to (129.0, 71.6)
- moved C19 47.8 mm to (132.1, 68.9), turned to 270 degrees
- moved C21 47.7 mm to (135.8, 116.8)
- moved C20 27.3 mm to (153.7, 88.9)
- moved R6 12.9 mm to (149.3, 150.0), turned to 90 degrees
- moved J3 11.0 mm to (112.0, 72.9)
- moved R1 8.72 mm to (112.5, 30.7), turned to 270 degrees
- moved SW5 7.67 mm to (149.9, 158.8)
- moved C29 7.39 mm to (151.1, 161.3)
- moved SW1 2.84 mm to (90.7, 153.5)
- moved SW2 2.84 mm to (86.7, 158.8)
- moved SW3 2.84 mm to (95.2, 158.8)
- moved SW4 2.84 mm to (90.7, 164.5)
- moved J12 1.05 mm to (109.0, 94.9)
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Connections:
- J14 pad 6: P0.07 -> P0.14
Routing:
- net GND: track 0.00 -> 685.3 mm, vias 0 -> 34
- net +3.3-SHIELD: track 0.00 -> 420.6 mm, vias 0 -> 24
- net P0.28: track 0.00 -> 126.9 mm, vias 0 -> 1
- net P0.25: track 0.00 -> 125.7 mm, vias 0 -> 5
- net Net-(B1-Pad3): track 0.00 -> 118.7 mm, vias 0 -> 3
- net P0.02: track 0.00 -> 115.5 mm, vias 0 -> 3
- net P0.27: track 0.00 -> 110.8 mm, vias 0 -> 1
- net P0.26: track 0.00 -> 90.6 mm, vias 0 -> 1
- net P0.10: track 0.00 -> 83.2 mm, vias 0 -> 4
- net P0.01: track 0.00 -> 79.8 mm
- net P0.06: track 0.00 -> 79.0 mm
- net P0.05: track 0.00 -> 78.0 mm
- net P0.07: track 0.00 -> 74.1 mm, vias 0 -> 3
- net P0.04: track 0.00 -> 72.7 mm, vias 0 -> 1
- net P0.09: track 0.00 -> 71.5 mm, vias 0 -> 3
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Other:
- board size 77.5 x 101.8 mm -> 77.5 x 142.5 mm
- board text added: "JOCO Badge Proto 1"

Commit message: layout maybe finished
Parts:
- removed J12: VBatt, Pin_Headers:Pin_Header_Straight_1x04_Pitch2.54mm
- removed J13: VBattSw, Pin_Headers:Pin_Header_Straight_1x04_Pitch2.54mm
- B1, R6: moved to B.Cu
- J1: footprint 1140084168:1140084168 -> sdcard:newsdcard
- moved B1 75.7 mm to (156.9, 119.4)
- moved BT1 71.4 mm to (155.8, 126.2), turned to 270 degrees
- moved J15 62.1 mm to (155.6, 146.1)
- moved C32 58.1 mm to (151.1, 144.9)
- moved L2 54.6 mm to (150.4, 139.6)
- moved U1 54.2 mm to (149.8, 135.2)
- moved C31 49.8 mm to (150.4, 130.6), turned to 180 degrees
- moved J2 20.4 mm to (142.9, 56.6)
- moved C30 9.66 mm to (140.4, 77.4), turned to 180 degrees
- moved C29 7.20 mm to (152.4, 154.2), turned to 180 degrees
- moved R7 4.92 mm to (136.4, 85.9)
- moved R6 3.91 mm to (147.2, 153.3)
- moved C1 3.60 mm to (99.4, 116.4)
- moved C2 2.25 mm to (99.4, 118.7), turned to 180 degrees
- moved L1 2.11 mm to (94.0, 133.6)
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Connections:
- BT1 pad 1: Net-(B1-Pad2) -> Net-(B1-Pad1)
- C31 pad 1: Net-(B1-Pad3) -> Net-(B1-Pad2)
- U1 pad 1: Net-(B1-Pad3) -> Net-(B1-Pad2)
- U1 pad 3: Net-(B1-Pad3) -> Net-(B1-Pad2)
Routing:
- net Net-(B1-Pad3): track 118.7 -> 0.00 mm, vias 3 -> 0
- net +3.3-SHIELD: track 420.6 -> 382.0 mm, vias 24 -> 22
- net Net-(D16-Pad2): track 32.7 -> 4.52 mm, vias 1 -> 0
- net P0.25: track 125.7 -> 151.8 mm, vias 5 -> 4
- net Net-(B1-Pad1): track 0.00 -> 18.0 mm
- net P0.27: track 110.8 -> 94.8 mm, vias 1 -> 2
- net Net-(B1-Pad2): track 36.8 -> 22.2 mm, vias 0 -> 3
- net P0.03: track 64.1 -> 49.8 mm
- net GND: track 685.3 -> 697.3 mm, vias 34 -> 31
- net P0.20: track 45.4 -> 52.8 mm
- net P0.08: track 47.8 -> 55.0 mm, vias 0 -> 3
- net P0.11: track 33.9 -> 40.0 mm, vias 0 -> 2
- net P0.19: track 33.7 -> 29.0 mm
- net +5-USB: track 48.9 -> 52.6 mm, vias 2 -> 1
- net P0.13: track 27.0 -> 30.5 mm
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Other:
- outline, holes or cut-outs redrawn
- board text added: "#badgelife"
- board text added: "+"
- board text added: "-"
