File: board/proto1/proto1.sch (KiCad schematic (older format))
At the start: 88 parts, among them J1 Micro_SD_Card_Det, J10 GND, J11 J11, J11A1 J11A, J12 VBatt, J13 VBattSw, J14 LCD, J15 3.3V Out, J2 LED_DOUT, J3 Expansion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

Commit message: lots more layout work
Parts:
- removed C23, C24: 0.1, Capacitors_SMD:C_0805, symbol C
- removed J11: J11, Pin_Headers:Pin_Header_Straight_2x03_Pitch2.54mm, symbol CONN_02X03
- removed J11A1: J11A, Pin_Headers:Pin_Header_Straight_2x03_Pitch2.54mm, symbol CONN_02X03
- removed J3: Expansion, Pin_Headers:Pin_Header_Straight_2x04_Pitch2.54mm, symbol CONN_02X04
- added J11: J11, Pin_Headers:Pin_Header_Straight_2x03_Pitch2.54mm, symbol Conn_02x03_Odd_Even
- added J11A1: J11A, Pin_Headers:Pin_Header_Straight_2x03_Pitch2.54mm, symbol Conn_02x03_Odd_Even
- added J3: Expansion, Pin_Headers:Pin_Header_Straight_2x04_Pitch2.54mm, symbol Conn_02x04_Odd_Even
- J10, J12, J13, J4: symbol CONN_01X04 -> Conn_01x04
- J14, J6, J6A1, J9, J9A1: symbol CONN_01X10 -> Conn_01x10
- J15: symbol CONN_01X02 -> Conn_01x02
- J2: symbol CONN_01X01 -> Conn_01x01
- J5, J5A1, J7, J7A1: symbol CONN_01X08 -> Conn_01x08
- J8, J8A1: symbol CONN_01X06 -> Conn_01x06
Connections:
- wire segments 327 -> 325

Commit message: layout maybe finished
Parts:
- removed J12: VBatt, Pin_Headers:Pin_Header_Straight_1x04_Pitch2.54mm, symbol Conn_01x04
- removed J13: VBattSw, Pin_Headers:Pin_Header_Straight_1x04_Pitch2.54mm, symbol Conn_01x04
- J1: footprint 1140084168:1140084168 -> sdcard:newsdcard
Connections:
- net at B1.1 (B): now also BT1.1 (+)
- net at B1.2 (COM): now also C31.1, U1.1 (VIN), U1.3 (~SHDN); no longer BT1.1 (+)
- now unconnected: B1.3 (A)
