File: board/proto2/badge.sch (EAGLE design)
At the start: 59 parts, among them IC1 TLV62569, J1 5051101092

Commit message: adding original AI from Amy; board specifications (TBD)
Other:
- note added: "".CMP" COMPONENT SIDE GERBER RS274X"
- note added: "".CRC" COMPONENT SIDE CREAM"
- note added: "".CRS" SOLDER SIDE CREAM"
- note added: "".DIM" DIMENSION LAYER WITH OUTSIDE DIMENSIONS IN MM"
- note added: "".DRD" EXCELLON DRILL FILE"
- note added: "".LY2" LAYER 2 GERBER RS274X"
- note added: "".LY3" LAYER 3 GERBER RS274X"
- note added: "".MIL" MILLING LAYER FOR INNER CUTOUTS (NOT PLATED)"
- note added: "".MNT" XYRS DATA FILE FOR PLACEMENT"
- note added: "".PLC" COMPONENT SIDE SILKSCREEN"
- note added: "".PLS" SOLDER SIDE SILKSCREEN"
- note added: "".SOL" SOLDER SIDE GERBER RS274X"
- note added: "".STC" COMPONENT SIDE SOLDER MASK STOP"
- note added: "".STS" SOLDER SIDE SOLDER MASK STOP"
- note added: "1-3u INCH OF GOLD OVER"
- note added: "1. THE PWB MUST BE LEAD FREE ASSEMBLY PROCESS COMPATIBLE"
- note added: "10. 15mil MAX RADIUS INSIDE MILLING CORNERS FOR SMALL RECTANGULAR OPENINGS"
- note added: "11. FILE DESIGNATIONS:"
- note added: "12. PLATED HOLE TOLERANCE .003""
- note added: "15 mil"
- note added: "2. PLATING FINISH - BOTH SIDES ENIG (ELECTROLESS NICKEL IMMERSION GOLD):"
- note added: "2.54-6.350 MICRON (100-250 MICROINCH) OF NICKEL."
- note added: "3. ALL THROUGH HOLE VIAS MAY BE PLATED SHUT"
- note added: "4. SOLDERMASK - BLACK COLOR, BOTH SIDES"
- note added: "5. SILKSCREEN - WHITE INK, BOTH SIDES. NO SILK ON PADS."
- note added: "6 mil"
- note added: "6. ELECTRICAL TEST - 100%"
- note added: "7. SUPPLIER MARKINGS - ALL MUST BE ON REAR OF PWB"
- note added: "8. MINIMUM CONDUCTIVE WIDTH/SPACING TO BE .004" / .004" EXCEPT IN DDR3 SIGNALS WHICH IS .004" / .0037""
- note added: "9. DIMENSIONAL OUTLINE OF PWB IN COMPONENT SILKSCREEN FILE"
- note added: "DIELECTRIC THICKNESSES"
- note added: "LAYER 1 - COMPONENT SIDE, 1oz FINISH"
- note added: "LAYER 2 - GROUND, 1/2oz"
- note added: "LAYER 3 - INNER SIGNAL LAYER, 1/2oz"
- note added: "LAYER 4 - GROUND , 1/2oz"
- note added: "LAYER 5 - POWER, 1/2oz"
- note added: "LAYER 6 - INNER SIGNAL LAYER, 1/2oz"
- note added: "LAYER 7 - GROUND, 1/2oz"
- note added: "LAYER 8 - SOLDER SIDE, 1oz FINISH"
- note added: "LAYER STACKUP DETAIL"
- note added: "NOTES (UNLESS OTHERWISE SPECIFIED)"
Changed lines of the file:
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@@
 <setting verticaltext="up"/>
 </settings>
-<grid distance="0.05" unitdist="inch" unit="inch" style="lines" multiple="1" display="no" altdistance="0.01" altunitdist="inch" altunit="inch"/>
+<grid distance="0.1" unitdist="inch" unit="inch" style="lines" multiple="1" display="no" altdistance="0.01" altunitdist="inch" altunit="inch"/>
 <layers>
 <layer number="1" name="Top" color="4" fill="1" visible="no" active="no"/>
@@
 <part name="SUPPLY32" library="supply2" deviceset="GND" device=""/>
 <part name="SUPPLY33" library="supply2" deviceset="GND" device=""/>
+<part name="FRAME1" library="frames" deviceset="FRAME_B_L" device="" value="21"/>
 </parts>
 <sheets>
@@
 </nets>
 </sheet>
+<sheet>
+<plain>
+<text x="340.36" y="26.67" size="1.778" layer="95">some statement of gracious attribution</text>
+<text x="358.14" y="31.75" size="1.778" layer="95">JoCo Badge</text>
+<wire x1="147.32" y1="53.34" x2="223.52" y2="53.34" width="1.27" layer="95"/>
+<wire x1="147.32" y1="7.62" x2="223.52" y2="7.62" width="1.27" layer="95"/>
+<wire x1="147.32" y1="12.7" x2="223.52" y2="12.7" width="0.6096" layer="95"/>
+<wire x1="147.32" y1="17.78" x2="223.52" y2="17.78" width="0.6096" layer="95"/>
+<wire x1="147.32" y1="27.94" x2="223.52" y2="27.94" width="0.6096" layer="95"/>
+<wire x1="147.32" y1="33.02" x2="223.52" y2="33.02" width="0.6096" layer="95"/>
+<wire x1="147.32" y1="43.18" x2="223.52" y2="43.18" width="0.6096" layer="95"/>
+<wire x1="147.32" y1="48.26" x2="223.52" y2="48.26" width="0.6096" layer="95"/>
+<text x="12.7" y="264.16" size="2.54" layer="95">NOTES (UNLESS OTHERWISE SPECIFIED)</text>
+<text x="17.78" y="259.08" size="2.54" layer="95">1. THE PWB MUST BE LEAD FREE ASSEMBLY PROCESS COMPATIBLE</text>
+<text x="17.78" y="254" size="2.54" layer="95">2. PLATING FINISH - BOTH SIDES ENIG (ELECTROLESS NICKEL IMMERSION GOLD):</text>
+<text x="40.64" y="248.92" size="2.54" layer="95">1-3u INCH OF GOLD OVER</text>
+<text x="40.64" y="243.84" size="2.54" layer="95">2.54-6.350 MICRON (100-250 MICROINCH) OF NICKEL.</text>
+<text x="17.78" y="238.76" size="2.54" layer="95">3. ALL THROUGH HOLE VIAS MAY BE PLATED SHUT</text>
+<text x="17.78" y="233.68" size="2.54" layer="95">4. SOLDERMASK - BLACK  COLOR, BOTH SIDES</text>
+<text x="17.78" y="228.6" size="2.54" layer="95">5. SILKSCREEN - WHITE INK, BOTH SIDES.  NO SILK ON PADS.</text>
+<text x="17.78" y="223.52" size="2.54" layer="95">6. ELECTRICAL TEST - 100%</text>
+<text x="17.78" y="218.44" size="2.54" layer="95">7. SUPPLIER MARKINGS - ALL MUST BE ON REAR OF PWB</text>
+<text x="17.78" y="213.36" size="2.54" layer="95">8. MINIMUM CONDUCTIVE WIDTH/SPACING TO BE .004" / .004" EXCEPT IN DDR3 SIGNALS WHICH IS .004" / .0037"</text>
+<text x="17.78" y="208.28" size="2.54" layer="95">9. DIMENSIONAL OUTLINE OF PWB IN COMPONENT SILKSCREEN FILE</text>
+<text x="17.78" y="198.12" size="2.54" layer="95">11. FILE DESIGNATIONS:</text>
+<text x="25.4" y="180.34" size="2.54" layer="95">".CMP"  COMPONENT SIDE GERBER RS274X</text>
+<text x="25.4" y="170.18" size="2.54" layer="95">".LY2"  LAYER 2 GERBER RS274X</text>
+<text x="25.4" y="165.1" size="2.54" layer="95">".LY3"  LAYER 3 GERBER RS274X</text>
+<text x="25.4" y="139.7" size="2.54" layer="95">".SOL"  SOLDER SIDE GERBER RS274X</text>
+<text x="25.4" y="190.5" size="2.54" layer="95">".PLC"  COMPONENT SIDE SILKSCREEN</text>
+<text x="25.4" y="129.54" size="2.54" layer="95">".PLS"  SOLDER SIDE SILKSCREEN</text>
+<text x="25.4" y="124.46" size="2.54" layer="95">".CRC"  COMPONENT SIDE CREAM</text>
+<text x="25.4" y="119.38" size="2.54" layer="95">".CRS"  SOLDER SIDE CREAM</text>
+<text x="25.4" y="185.42" size="2.54" layer="95">".STC"  COMPONENT SIDE SOLDER MASK STOP</text>
+<text x="25.4" y="134.62" size="2.54" layer="95">".STS"  SOLDER SIDE SOLDER MASK STOP</text>
+<text x="25.4" y="109.22" size="2.54" layer="95">".DRD"  EXCELLON DRILL FILE</text>
+<text x="25.4" y="104.14" size="2.54" layer="95">".MNT"  XYRS DATA FILE FOR PLACEMENT</text>
+<text x="229.87" y="52.07" size="2.54" layer="95">LAYER 1 - COMPONENT SIDE, 1oz FINISH</text>
+<text x="229.87" y="46.99" size="2.54" layer="95">LAYER 2 - GROUND, 1/2oz</text>
+<text x="229.87" y="41.91" size="2.54" layer="95">LAYER 3 - INNER SIGNAL LAYER, 1/2oz</text>
+<text x="229.87" y="31.75" size="2.54" layer="95">LAYER 4 - GROUND , 1/2oz</text>
+<text x="229.87" y="26.67" size="2.54" layer="95">LAYER 5 - POWER, 1/2oz</text>
+<text x="229.87" y="16.51" size="2.54" layer="95">LAYER 6 - INNER SIGNAL LAYER, 1/2oz</text>
+<text x="229.87" y="11.43" size="2.54" layer="95">LAYER 7 - GROUND, 1/2oz</text>
+<text x="229.87" y="6.35" size="2.54" layer="95">LAYER 8 - SOLDER SIDE, 1oz FINISH</text>
+<text x="101.219" y="36.957" size="2.54" layer="95">DIELECTRIC THICKNESSES</text>
+<text x="181.61" y="49.53" size="2.1844" layer="95">6 mil</text>
+<text x="181.61" y="8.89" size="2.1844" layer="95">6 mil</text>
+<text x="181.61" y="44.45" size="2.1844" layer="95">6 mil</text>
+<text x="181.61" y="29.21" size="2.1844" layer="95">6 mil</text>
+<text x="181.61" y="13.97" size="2.1844" layer="95">6 mil</text>
+<text x="180.34" y="36.83" size="2.1844" layer="95">15 mil</text>
+<text x="180.34" y="21.59" size="2.1844" layer="95">15 mil</text>
+<text x="161.417" y="63.119" size="3.175" layer="95">LAYER STACKUP DETAIL</text>
+<text x="16.51" y="97.79" size="2.54" layer="95">12. PLATED HOLE TOLERANCE  .003"</text>
+<text x="25.4" y="114.3" size="2.54" layer="97">".MIL"  MILLING LAYER FOR INNER CUTOUTS (NOT PLATED)</text>
+<text x="17.78" y="203.2" size="2.54" layer="95">10. 15mil MAX RADIUS  INSIDE MILLING CORNERS FOR SMALL RECTANGULAR OPENINGS</text>
+<text x="25.4" y="175.26" size="2.54" layer="95">".DIM"  DIMENSION LAYER WITH OUTSIDE DIMENSIONS IN MM</text>
+</plain>
+<instances>
+<instance part="FRAME1" gate="G$1" x="0" y="0"/>
+<instance part="FRAME1" gate="G$2" x="325.12" y="0"/>
+</instances>
+<busses>
+</busses>
+<nets>
+</nets>
+</sheet>

Commit message: reduce LEDs to 14, add tilt switch, draw NFC antenna
Parts:
- removed C19, C23: .1u, rcl:C-USC0201
- removed LED15, LED16: WS2812B, badge:WS2812B
- added S7: SW-200D, badge:SW-200D
Connections:
- removed net N$26: LED15.DOUT, LED16.DIN
- net +3V3: no longer C19.1, C23.1, LED15.VDD, LED16.VDD
- net GND: now also S7.P$1; no longer C19.2, C23.2, LED15.VSS, LED16.VSS
- net N$21: now also S7.P$2, U1.P0.19; no longer LED14.DOUT, LED15.DIN
Other:
- note added: "TILT SWITCH"
Changed lines of the file:
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@@
 <setting verticaltext="up"/>
 </settings>
-<grid distance="0.1" unitdist="inch" unit="inch" style="lines" multiple="1" display="no" altdistance="0.01" altunitdist="inch" altunit="inch"/>
+<grid distance="0.05" unitdist="inch" unit="inch" style="lines" multiple="1" display="no" altdistance="0.01" altunitdist="inch" altunit="inch"/>
 <layers>
 <layer number="1" name="Top" color="4" fill="1" visible="no" active="no"/>
@@
 <part name="LED13" library="badge" deviceset="WS2812B" device=""/>
 <part name="LED14" library="badge" deviceset="WS2812B" device=""/>
-<part name="LED15" library="badge" deviceset="WS2812B" device=""/>
-<part name="LED16" library="badge" deviceset="WS2812B" device=""/>
 <part name="SUPPLY14" library="supply2" deviceset="GND" device=""/>
 <part name="SUPPLY15" library="supply2" deviceset="GND" device=""/>
@@
 <part name="C17" library="rcl" deviceset="C-US" device="C0201" value=".1u"/>
 <part name="C18" library="rcl" deviceset="C-US" device="C0201" value=".1u"/>
-<part name="C19" library="rcl" deviceset="C-US" device="C0201" value=".1u"/>
 <part name="C20" library="rcl" deviceset="C-US" device="C0201" value=".1u"/>
 <part name="C21" library="rcl" deviceset="C-US" device="C0201" value=".1u"/>
 <part name="C22" library="rcl" deviceset="C-US" device="C0201" value=".1u"/>
-<part name="C23" library="rcl" deviceset="C-US" device="C0201" value=".1u"/>
 <part name="SUPPLY26" library="supply2" deviceset="GND" device=""/>
 <part name="SUPPLY27" library="supply2" deviceset="GND" device=""/>
 <part name="SUPPLY28" library="supply2" deviceset="GND" device=""/>
-<part name="SUPPLY29" library="supply2" deviceset="GND" device=""/>
 <part name="SUPPLY30" library="supply2" deviceset="GND" device=""/>
 <part name="SUPPLY31" library="supply2" deviceset="GND" device=""/>
 <part name="SUPPLY32" library="supply2" deviceset="GND" device=""/>
-<part name="SUPPLY33" library="supply2" deviceset="GND" device=""/>
 <part name="FRAME1" library="frames" deviceset="FRAME_B_L" device="" value="21"/>
+<part name="S7" library="badge" deviceset="SW-200D" device=""/>
+<part name="SUPPLY29" library="supply2" deviceset="GND" device=""/>
 </parts>
 <sheets>
@@
 <text x="86.36" y="176.53" size="1.27" layer="98">DOWN</text>
 <text x="86.36" y="168.91" size="1.27" layer="98">ACTION</text>
+<text x="246.38" y="132.08" size="1.778" layer="97" rot="R90">TILT SWITCH</text>
 </plain>
 <instances>
@@
 <instance part="LED13" gate="G$1" x="276.86" y="182.88"/>
 <instance part="LED14" gate="G$1" x="314.96" y="182.88"/>
-<instance part="LED15" gate="G$1" x="353.06" y="182.88"/>
-<instance part="LED16" gate="G$1" x="391.16" y="182.88"/>
 <instance part="SUPPLY14" gate="GND" x="292.1" y="167.64"/>
 <instance part="SUPPLY15" gate="GND" x="330.2" y="167.64"/>
@@
 <instance part="C17" gate="G$1" x="351.79" y="153.67" rot="MR0"/>
 <instance part="C18" gate="G$1" x="359.41" y="153.67" rot="MR0"/>
-<instance part="C19" gate="G$1" x="367.03" y="153.67" rot="MR0"/>
 <instance part="C20" gate="G$1" x="379.73" y="153.67" rot="MR0"/>
 <instance part="C21" gate="G$1" x="387.35" y="153.67" rot="MR0"/>
 <instance part="C22" gate="G$1" x="394.97" y="153.67" rot="MR0"/>
-<instance part="C23" gate="G$1" x="402.59" y="153.67" rot="MR0"/>
 <instance part="SUPPLY26" gate="GND" x="344.17" y="146.05"/>
 <instance part="SUPPLY27" gate="GND" x="351.79" y="146.05"/>
 <instance part="SUPPLY28" gate="GND" x="359.41" y="146.05"/>
-<instance part="SUPPLY29" gate="GND" x="367.03" y="146.05"/>
 <instance part="SUPPLY30" gate="GND" x="379.73" y="146.05"/>
 <instance part="SUPPLY31" gate="GND" x="387.35" y="146.05"/>
 <instance part="SUPPLY32" gate="GND" x="394.97" y="146.05"/>
-<instance part="SUPPLY33" gate="GND" x="402.59" y="146.05"/>
+<instance part="S7" gate="G$1" x="238.76" y="139.7" rot="R90"/>
+<instance part="SUPPLY29" gate="GND" x="238.76" y="124.46"/>
 </instances>
 <busses>
@@
 <wire x1="365.76" y1="241.3" x2="368.3" y2="241.3" width="0.1524" layer="91"/>
 <wire x1="368.3" y1="241.3" x2="368.3" y2="220.98" width="0.1524" layer="91"/>
-<pinref part="LED15" gate="G$1" pin="VSS"/>
 <wire x1="368.3" y1="220.98" x2="368.3" y2="200.66" width="0.1524" layer="91"/>
-<wire x1="368.3" y1="200.66" x2="368.3" y2="180.34" width="0.1524" layer="91"/>
-<wire x1="368.3" y1="180.34" x2="368.3" y2="170.18" width="0.1524" layer="91"/>
-<wire x1="365.76" y1="180.34" x2="368.3" y2="180.34" width="0.1524" layer="91"/>
-<junction x="368.3" y="180.34"/>
+<wire x1="368.3" y1="200.66" x2="368.3" y2="170.18" width="0.1524" layer="91"/>
 <pinref part="LED11" gate="G$1" pin="VSS"/>
 <wire x1="365.76" y1="200.66" x2="368.3" y2="200.66" width="0.1524" layer="91"/>
@@
 <wire x1="403.86" y1="241.3" x2="406.4" y2="241.3" width="0.1524" layer="91"/>
 <wire x1="406.4" y1="241.3" x2="406.4" y2="220.98" width="0.1524" layer="91"/>
-<pinref part="LED16" gate="G$1" pin="VSS"/>
 <wire x1="406.4" y1="220.98" x2="406.4" y2="200.66" width="0.1524" layer="91"/>
-<wire x1="406.4" y1="200.66" x2="406.4" y2="180.34" width="0.1524" layer="91"/>
-<wire x1="406.4" y1="180.34" x2="406.4" y2="170.18" width="0.1524" layer="91"/>
-<wire x1="403.86" y1="180.34" x2="406.4" y2="180.34" width="0.1524" layer="91"/>
-<junction x="406.4" y="180.34"/>
+<wire x1="406.4" y1="200.66" x2="406.4" y2="170.18" width="0.1524" layer="91"/>
 <pinref part="LED12" gate="G$1" pin="VSS"/>
 <wire x1="403.86" y1="200.66" x2="406.4" y2="200.66" width="0.1524" layer="91"/>
@@
 </segment>
 <segment>
-<pinref part="C19" gate="G$1" pin="2"/>
-<pinref part="SUPPLY29" gate="GND" pin="GND"/>
-</segment>
-<segment>
 <pinref part="C20" gate="G$1" pin="2"/>
 <pinref part="SUPPLY30" gate="GND" pin="GND"/>
@@
 </segment>
 <segment>
-<pinref part="C23" gate="G$1" pin="2"/>
-<pinref part="SUPPLY33" gate="GND" pin="GND"/>
+<pinref part="S7" gate="G$1" pin="P$1"/>
+<wire x1="238.76" y1="129.54" x2="238.76" y2="127" width="0.1524" layer="91"/>
+<pinref part="SUPPLY29" gate="GND" pin="GND"/>
 </segment>
 </net>
@@
 </segment>
 <segment>
-<pinref part="LED15" gate="G$1" pin="VDD"/>
-<wire x1="342.9" y1="185.42" x2="340.36" y2="185.42" width="0.1524" layer="91"/>
-<wire x1="340.36" y1="185.42" x2="340.36" y2="205.74" width="0.1524" layer="91"/>
 <pinref part="LED3" gate="G$1" pin="VDD"/>
 <wire x1="340.36" y1="205.74" x2="340.36" y2="226.06" width="0.1524" layer="91"/>
@@
 <wire x1="359.41" y1="158.75" x2="359.41" y2="156.21" width="0.1524" layer="91"/>
 <junction x="351.79" y="158.75"/>
-<pinref part="C19" gate="G$1" pin="1"/>
-<wire x1="359.41" y1="158.75" x2="367.03" y2="158.75" width="0.1524" layer="91"/>
-<wire x1="367.03" y1="158.75" x2="367.03" y2="156.21" width="0.1524" layer="91"/>
-<junction x="359.41" y="158.75"/>
 <wire x1="344.17" y1="158.75" x2="340.36" y2="158.75" width="0.1524" layer="91"/>
-<wire x1="340.36" y1="158.75" x2="340.36" y2="185.42" width="0.1524" layer="91"/>
+<wire x1="340.36" y1="158.75" x2="340.36" y2="205.74" width="0.1524" layer="91"/>
 <junction x="344.17" y="158.75"/>
-<junction x="340.36" y="185.42"/>
-</segment>
-<segment>
-<pinref part="LED16" gate="G$1" pin="VDD"/>
-<wire x1="381" y1="185.42" x2="378.46" y2="185.42" width="0.1524" layer="91"/>
-<wire x1="378.46" y1="185.42" x2="378.46" y2="205.74" width="0.1524" layer="91"/>
+</segment>
+<segment>
 <pinref part="LED4" gate="G$1" pin="VDD"/>
 <wire x1="378.46" y1="205.74" x2="378.46" y2="226.06" width="0.1524" layer="91"/>
@@
 <wire x1="394.97" y1="158.75" x2="394.97" y2="156.21" width="0.1524" layer="91"/>
 <junction x="387.35" y="158.75"/>
-<pinref part="C23" gate="G$1" pin="1"/>
-<wire x1="394.97" y1="158.75" x2="402.59" y2="158.75" width="0.1524" layer="91"/>
-<wire x1="402.59" y1="158.75" x2="402.59" y2="156.21" width="0.1524" layer="91"/>
-<junction x="394.97" y="158.75"/>
 <wire x1="379.73" y1="158.75" x2="378.46" y2="158.75" width="0.1524" layer="91"/>
-<wire x1="378.46" y1="158.75" x2="378.46" y2="185.42" width="0.1524" layer="91"/>
+<wire x1="378.46" y1="158.75" x2="378.46" y2="205.74" width="0.1524" layer="91"/>
 <junction x="379.73" y="158.75"/>
-<junction x="378.46" y="185.42"/>
 </segment>
 </net>
@@
 </segment>
 </net>
-<net name="N$21" class="0">
-<segment>
-<pinref part="LED14" gate="G$1" pin="DOUT"/>
-<wire x1="327.66" y1="185.42" x2="332.74" y2="185.42" width="0.1524" layer="91"/>
-<wire x1="332.74" y1="185.42" x2="337.82" y2="180.34" width="0.1524" layer="91"/>
-<pinref part="LED15" gate="G$1" pin="DIN"/>
-<wire x1="337.82" y1="180.34" x2="342.9" y2="180.34" width="0.1524" layer="91"/>
-</segment>
-</net>
 <net name="N$22" class="0">
 <segment>
@@
 <pinref part="LED12" gate="G$1" pin="DIN"/>
 <wire x1="375.92" y1="200.66" x2="381" y2="200.66" width="0.1524" layer="91"/>
-</segment>
-</net>
-<net name="N$26" class="0">
-<segment>
-<pinref part="LED15" gate="G$1" pin="DOUT"/>
-<wire x1="365.76" y1="185.42" x2="370.84" y2="185.42" width="0.1524" layer="91"/>
-<wire x1="370.84" y1="185.42" x2="375.92" y2="180.34" width="0.1524" layer="91"/>
-<pinref part="LED16" gate="G$1" pin="DIN"/>
-<wire x1="375.92" y1="180.34" x2="381" y2="180.34" width="0.1524" layer="91"/>
 </segment>
 </net>
@@
 </segment>
 </net>
+<net name="N$21" class="0">
+<segment>
+<pinref part="S7" gate="G$1" pin="P$2"/>
+<wire x1="238.76" y1="175.26" x2="238.76" y2="149.86" width="0.1524" layer="91"/>
+<pinref part="U1" gate="G$1" pin="P0.19"/>
+<wire x1="213.36" y1="175.26" x2="238.76" y2="175.26" width="0.1524" layer="91"/>
+</segment>
+</net>
