File: board/proto2/badge.sch (EAGLE design)
At the start: 67 parts, among them IC1 TLV62569, J1 5051101092, J2 M05X2X1.27

Commit message: lots of routing going on
Parts:
- removed C21, C22: .1u, rcl:C-USC0402K
Connections:
- net N$14 renamed SW
- net N$21 renamed P0.19
- net N$26 renamed SWDIO
- net N$31 renamed SWCLK
- net N$32 renamed P0.18
- net N$33 renamed !RESET
- net +3V3: no longer C21.1, C22.1
- net GND: no longer C21.2, C22.2
Other:
- moved on the sheet: C20
Changed lines of the file:
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@@
 <part name="C16" library="rcl" deviceset="C-US" device="C0402K" value=".1u"/>
 <part name="C17" library="rcl" deviceset="C-US" device="C0402K" value=".1u"/>
-<part name="C18" library="rcl" deviceset="C-US" device="C0402K" value=".1u"/>
-<part name="C20" library="rcl" deviceset="C-US" device="C0402K" value=".1u"/>
-<part name="C21" library="rcl" deviceset="C-US" device="C0402K" value=".1u"/>
-<part name="C22" library="rcl" deviceset="C-US" device="C0402K" value=".1u"/>
 <part name="SUPPLY26" library="supply2" deviceset="GND" device=""/>
 <part name="SUPPLY27" library="supply2" deviceset="GND" device=""/>
-<part name="SUPPLY28" library="supply2" deviceset="GND" device=""/>
-<part name="SUPPLY30" library="supply2" deviceset="GND" device=""/>
-<part name="SUPPLY31" library="supply2" deviceset="GND" device=""/>
-<part name="SUPPLY32" library="supply2" deviceset="GND" device=""/>
 <part name="FRAME1" library="frames" deviceset="FRAME_B_L" device="" value="21"/>
 <part name="S7" library="badge" deviceset="SW-200D" device=""/>
@@
 <part name="C28" library="rcl" deviceset="C-US" device="C0402K" value=".1u"/>
 <part name="OLED1" library="badge" deviceset="CFAF128128B" device=""/>
+<part name="C18" library="rcl" deviceset="C-US" device="C0402K" value=".1u"/>
+<part name="SUPPLY28" library="supply2" deviceset="GND" device=""/>
+<part name="C20" library="rcl" deviceset="C-US" device="C0402K" value=".1u"/>
+<part name="SUPPLY30" library="supply2" deviceset="GND" device=""/>
 </parts>
 <sheets>
@@
 <instance part="C16" gate="G$1" x="344.17" y="153.67" rot="MR0"/>
 <instance part="C17" gate="G$1" x="351.79" y="153.67" rot="MR0"/>
-<instance part="C18" gate="G$1" x="359.41" y="153.67" rot="MR0"/>
-<instance part="C20" gate="G$1" x="379.73" y="153.67" rot="MR0"/>
-<instance part="C21" gate="G$1" x="387.35" y="153.67" rot="MR0"/>
-<instance part="C22" gate="G$1" x="394.97" y="153.67" rot="MR0"/>
 <instance part="SUPPLY26" gate="GND" x="344.17" y="146.05"/>
 <instance part="SUPPLY27" gate="GND" x="351.79" y="146.05"/>
-<instance part="SUPPLY28" gate="GND" x="359.41" y="146.05"/>
-<instance part="SUPPLY30" gate="GND" x="379.73" y="146.05"/>
-<instance part="SUPPLY31" gate="GND" x="387.35" y="146.05"/>
-<instance part="SUPPLY32" gate="GND" x="394.97" y="146.05"/>
 <instance part="S7" gate="G$1" x="238.76" y="139.7" rot="R90"/>
 <instance part="SUPPLY29" gate="GND" x="238.76" y="124.46"/>
@@
 <instance part="C28" gate="G$1" x="204.47" y="220.98" rot="MR0"/>
 <instance part="OLED1" gate="G$1" x="128.27" y="241.3"/>
+<instance part="C18" gate="G$1" x="359.41" y="153.67" rot="MR0"/>
+<instance part="SUPPLY28" gate="GND" x="359.41" y="146.05"/>
+<instance part="C20" gate="G$1" x="367.03" y="153.67" rot="MR0"/>
+<instance part="SUPPLY30" gate="GND" x="367.03" y="146.05"/>
 </instances>
 <busses>
@@
 </segment>
 <segment>
-<pinref part="C18" gate="G$1" pin="2"/>
-<pinref part="SUPPLY28" gate="GND" pin="GND"/>
-</segment>
-<segment>
-<pinref part="C20" gate="G$1" pin="2"/>
-<pinref part="SUPPLY30" gate="GND" pin="GND"/>
-</segment>
-<segment>
-<pinref part="C21" gate="G$1" pin="2"/>
-<pinref part="SUPPLY31" gate="GND" pin="GND"/>
-</segment>
-<segment>
-<pinref part="C22" gate="G$1" pin="2"/>
-<pinref part="SUPPLY32" gate="GND" pin="GND"/>
-</segment>
-<segment>
 <pinref part="S7" gate="G$1" pin="P$1"/>
 <wire x1="238.76" y1="129.54" x2="238.76" y2="127" width="0.1524" layer="91"/>
@@
 <pinref part="C28" gate="G$1" pin="2"/>
 <pinref part="SUPPLY42" gate="GND" pin="GND"/>
+</segment>
+<segment>
+<pinref part="C18" gate="G$1" pin="2"/>
+<pinref part="SUPPLY28" gate="GND" pin="GND"/>
+</segment>
+<segment>
+<pinref part="C20" gate="G$1" pin="2"/>
+<pinref part="SUPPLY30" gate="GND" pin="GND"/>
 </segment>
 </net>
@@
 <wire x1="344.17" y1="158.75" x2="351.79" y2="158.75" width="0.1524" layer="91"/>
 <wire x1="351.79" y1="158.75" x2="351.79" y2="156.21" width="0.1524" layer="91"/>
-<pinref part="C18" gate="G$1" pin="1"/>
-<wire x1="351.79" y1="158.75" x2="359.41" y2="158.75" width="0.1524" layer="91"/>
-<wire x1="359.41" y1="158.75" x2="359.41" y2="156.21" width="0.1524" layer="91"/>
-<junction x="351.79" y="158.75"/>
 <wire x1="344.17" y1="158.75" x2="340.36" y2="158.75" width="0.1524" layer="91"/>
 <wire x1="340.36" y1="158.75" x2="340.36" y2="205.74" width="0.1524" layer="91"/>
 <junction x="344.17" y="158.75"/>
+<wire x1="351.79" y1="158.75" x2="359.41" y2="158.75" width="0.1524" layer="91"/>
+<junction x="351.79" y="158.75"/>
+<pinref part="C18" gate="G$1" pin="1"/>
+<wire x1="359.41" y1="158.75" x2="359.41" y2="156.21" width="0.1524" layer="91"/>
+<wire x1="359.41" y1="158.75" x2="367.03" y2="158.75" width="0.1524" layer="91"/>
+<junction x="359.41" y="158.75"/>
+<pinref part="C20" gate="G$1" pin="1"/>
+<wire x1="367.03" y1="158.75" x2="367.03" y2="156.21" width="0.1524" layer="91"/>
 </segment>
 <segment>
@@
 <pinref part="LED12" gate="G$1" pin="VDD"/>
 <wire x1="381" y1="205.74" x2="378.46" y2="205.74" width="0.1524" layer="91"/>
-<junction x="378.46" y="205.74"/>
 <pinref part="+3V6" gate="G$1" pin="+3V3"/>
-<pinref part="C20" gate="G$1" pin="1"/>
-<wire x1="379.73" y1="156.21" x2="379.73" y2="158.75" width="0.1524" layer="91"/>
-<pinref part="C21" gate="G$1" pin="1"/>
-<wire x1="379.73" y1="158.75" x2="387.35" y2="158.75" width="0.1524" layer="91"/>
-<wire x1="387.35" y1="158.75" x2="387.35" y2="156.21" width="0.1524" layer="91"/>
-<pinref part="C22" gate="G$1" pin="1"/>
-<wire x1="387.35" y1="158.75" x2="394.97" y2="158.75" width="0.1524" layer="91"/>
-<wire x1="394.97" y1="158.75" x2="394.97" y2="156.21" width="0.1524" layer="91"/>
-<junction x="387.35" y="158.75"/>
-<wire x1="379.73" y1="158.75" x2="378.46" y2="158.75" width="0.1524" layer="91"/>
-<wire x1="378.46" y1="158.75" x2="378.46" y2="205.74" width="0.1524" layer="91"/>
-<junction x="379.73" y="158.75"/>
 </segment>
 <segment>
@@
 </segment>
 </net>
-<net name="N$14" class="0">
+<net name="SW" class="0">
 <segment>
 <pinref part="IC1" gate="G$1" pin="SW"/>
@@
 </segment>
 </net>
-<net name="N$21" class="0">
+<net name="P0.19" class="0">
 <segment>
 <pinref part="S7" gate="G$1" pin="P$2"/>
@@
 </segment>
 </net>
-<net name="N$26" class="0">
+<net name="SWDIO" class="0">
 <segment>
 <pinref part="J2" gate="G$1" pin="2"/>
@@
 </segment>
 </net>
-<net name="N$31" class="0">
+<net name="SWCLK" class="0">
 <segment>
 <pinref part="J2" gate="G$1" pin="4"/>
@@
 </segment>
 </net>
-<net name="N$32" class="0">
+<net name="P0.18" class="0">
 <segment>
 <pinref part="J2" gate="G$1" pin="6"/>
@@
 </segment>
 </net>
-<net name="N$33" class="0">
+<net name="!RESET" class="0">
 <segment>
 <pinref part="J2" gate="G$1" pin="10"/>

Commit message: remove unneeded pin labels
Parts:
- JP1: value (none) -> NP
- U1: value (none) -> BMD-300
Connections:
- removed net P0.15: U1.TRACED[2]/P0.15
- removed net P0.16: U1.TRACED[1]/P0.16
Changed lines of the file:
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@@
 </classes>
 <parts>
-<part name="U1" library="BMD-300" deviceset="BMD-300" device=""/>
+<part name="U1" library="BMD-300" deviceset="BMD-300" device="" value="BMD-300"/>
 <part name="FRAME13" library="frames" deviceset="FRAME_B_L" device="" value="21"/>
 <part name="B1" library="badge" deviceset="12BH331P-GR" device=""/>
@@
 <part name="SUPPLY35" library="supply2" deviceset="GND" device=""/>
 <part name="+3V7" library="supply1" deviceset="+3V3" device=""/>
-<part name="JP1" library="pinhead" deviceset="PINHD-2X4" device=""/>
+<part name="JP1" library="pinhead" deviceset="PINHD-2X4" device="" value="NP"/>
 <part name="+3V8" library="supply1" deviceset="+3V3" device=""/>
 <part name="SUPPLY36" library="supply2" deviceset="GND" device=""/>
@@
 <text x="246.38" y="132.08" size="1.778" layer="97" rot="R90">TILT SWITCH</text>
 <text x="190.5" y="95.25" size="1.778" layer="97">NFC ANTENNA</text>
-<text x="64.77" y="99.06" size="1.778" layer="97">EXPANSION</text>
+<text x="63.5" y="96.52" size="1.778" layer="97">EXPANSION</text>
 <text x="223.52" y="232.41" size="1.778" layer="97">PROGRAM</text>
 </plain>
@@
 </segment>
 </net>
-<net name="P0.15" class="0">
-<segment>
-<pinref part="U1" gate="G$1" pin="TRACED[2]/P0.15"/>
-<wire x1="213.36" y1="165.1" x2="220.98" y2="165.1" width="0.1524" layer="91"/>
-<label x="220.98" y="165.1" size="1.27" layer="91" xref="yes"/>
-</segment>
-</net>
-<net name="P0.16" class="0">
-<segment>
-<pinref part="U1" gate="G$1" pin="TRACED[1]/P0.16"/>
-<wire x1="213.36" y1="167.64" x2="220.98" y2="167.64" width="0.1524" layer="91"/>
-<label x="220.98" y="167.64" size="1.27" layer="91" xref="yes"/>
-</segment>
-</net>
-<net name="P0.17" class="0">
-<segment>
-<wire x1="214.63" y1="170.18" x2="220.98" y2="170.18" width="0.1524" layer="91"/>
-<label x="220.98" y="170.18" size="1.27" layer="91" xref="yes"/>
-</segment>
-</net>

Commit message: changes for errors found by AI4QR
Parts:
- added C21: .1u, rcl:C-USC0402K
- added R10: 1.0k, rcl:R-US_R0603
- R8: value 47 -> 220
Connections:
- new net N$11: C21.1, R10.1, S7.P$2
- net GND: now also C21.2
- net P0.19: now also R10.2; no longer S7.P$2

Commit message: final changes to proto2, saving Gerbers
Parts:
- B1: value 12BH331P-GR -> 2464; device badge:12BH331P-GR -> badge:2464
Other:
- note added: "60 mil"
- note added: "LAYER 2 - SOLDER SIDE, 1oz FINISH"
- note removed: "".LY2" LAYER 2 GERBER RS274X"
- note removed: "".LY3" LAYER 3 GERBER RS274X"
- note removed: "15 mil"
- note removed: "6 mil"
- note removed: "LAYER 2 - GROUND, 1/2oz"
- note removed: "LAYER 3 - INNER SIGNAL LAYER, 1/2oz"
- note removed: "LAYER 4 - GROUND , 1/2oz"
- note removed: "LAYER 5 - POWER, 1/2oz"
- note removed: "LAYER 6 - INNER SIGNAL LAYER, 1/2oz"
- note removed: "LAYER 7 - GROUND, 1/2oz"
- note removed: "LAYER 8 - SOLDER SIDE, 1oz FINISH"
Changed lines of the file:
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@@
 <setting verticaltext="up"/>
 </settings>
-<grid distance="0.05" unitdist="inch" unit="inch" style="lines" multiple="1" display="no" altdistance="0.01" altunitdist="inch" altunit="inch"/>
+<grid distance="0.1" unitdist="inch" unit="inch" style="lines" multiple="1" display="no" altdistance="0.01" altunitdist="inch" altunit="inch"/>
 <layers>
 <layer number="1" name="Top" color="4" fill="1" visible="no" active="no"/>
@@
 <part name="U1" library="BMD-300" deviceset="BMD-300" device="" value="BMD-300"/>
 <part name="FRAME13" library="frames" deviceset="FRAME_B_L" device="" value="21"/>
-<part name="B1" library="badge" deviceset="12BH331P-GR" device=""/>
 <part name="S1" library="badge" deviceset="PTS810" device=""/>
 <part name="S2" library="badge" deviceset="PTS810" device=""/>
@@
 <part name="C21" library="rcl" deviceset="C-US" device="C0402K" value=".1u"/>
 <part name="SUPPLY31" library="supply2" deviceset="GND" device=""/>
+<part name="B1" library="badge" deviceset="2464" device=""/>
 </parts>
 <sheets>
@@
 <instance part="FRAME13" gate="G$1" x="0" y="0"/>
 <instance part="FRAME13" gate="G$2" x="325.12" y="0"/>
-<instance part="B1" gate="G$1" x="22.86" y="241.3" smashed="yes" rot="R90">
-<attribute name="NAME" x="19.05" y="237.49" size="1.778" layer="95" rot="R90"/>
-<attribute name="VALUE" x="17.78" y="245.11" size="1.778" layer="96" rot="R90"/>
-</instance>
 <instance part="S1" gate="G$1" x="83.82" y="195.58" smashed="yes">
 <attribute name="NAME" x="80.01" y="199.39" size="1.27" layer="95"/>
@@
 <instance part="C21" gate="G$1" x="259.08" y="146.05" rot="MR0"/>
 <instance part="SUPPLY31" gate="GND" x="259.08" y="138.43"/>
+<instance part="B1" gate="G$1" x="22.86" y="241.3" rot="R90"/>
 </instances>
 <busses>
@@
 <wire x1="41.91" y1="238.76" x2="29.21" y2="238.76" width="0.1524" layer="91"/>
 <wire x1="29.21" y1="238.76" x2="29.21" y2="231.14" width="0.1524" layer="91"/>
-<pinref part="B1" gate="G$1" pin="-"/>
 <wire x1="29.21" y1="231.14" x2="29.21" y2="228.6" width="0.1524" layer="91"/>
 <wire x1="22.86" y1="233.68" x2="22.86" y2="231.14" width="0.1524" layer="91"/>
@@
 <junction x="29.21" y="231.14"/>
 <pinref part="SUPPLY8" gate="GND" pin="GND"/>
+<pinref part="B1" gate="G$1" pin="-"/>
 </segment>
 <segment>
@@
 <net name="VIN" class="0">
 <segment>
-<pinref part="B1" gate="G$1" pin="+"/>
 <pinref part="S6" gate="G$1" pin="3"/>
 <wire x1="22.86" y1="248.92" x2="22.86" y2="264.16" width="0.1524" layer="91"/>
 <wire x1="22.86" y1="264.16" x2="24.13" y2="264.16" width="0.1524" layer="91"/>
+<pinref part="B1" gate="G$1" pin="+"/>
 </segment>
 </net>
@@
 <wire x1="147.32" y1="53.34" x2="223.52" y2="53.34" width="1.27" layer="95"/>
 <wire x1="147.32" y1="7.62" x2="223.52" y2="7.62" width="1.27" layer="95"/>
-<wire x1="147.32" y1="12.7" x2="223.52" y2="12.7" width="0.6096" layer="95"/>
-<wire x1="147.32" y1="17.78" x2="223.52" y2="17.78" width="0.6096" layer="95"/>
-<wire x1="147.32" y1="27.94" x2="223.52" y2="27.94" width="0.6096" layer="95"/>
-<wire x1="147.32" y1="33.02" x2="223.52" y2="33.02" width="0.6096" layer="95"/>
-<wire x1="147.32" y1="43.18" x2="223.52" y2="43.18" width="0.6096" layer="95"/>
-<wire x1="147.32" y1="48.26" x2="223.52" y2="48.26" width="0.6096" layer="95"/>
 <text x="12.7" y="264.16" size="2.54" layer="95">NOTES (UNLESS OTHERWISE SPECIFIED)</text>
 <text x="17.78" y="259.08" size="2.54" layer="95">1. THE PWB MUST BE LEAD FREE ASSEMBLY PROCESS COMPATIBLE</text>
@@
 <text x="17.78" y="198.12" size="2.54" layer="95">11. FILE DESIGNATIONS:</text>
 <text x="25.4" y="180.34" size="2.54" layer="95">".CMP"  COMPONENT SIDE GERBER RS274X</text>
-<text x="25.4" y="170.18" size="2.54" layer="95">".LY2"  LAYER 2 GERBER RS274X</text>
-<text x="25.4" y="165.1" size="2.54" layer="95">".LY3"  LAYER 3 GERBER RS274X</text>
-<text x="25.4" y="139.7" size="2.54" layer="95">".SOL"  SOLDER SIDE GERBER RS274X</text>
+<text x="25.4" y="170.18" size="2.54" layer="95">".SOL"  SOLDER SIDE GERBER RS274X</text>
 <text x="25.4" y="190.5" size="2.54" layer="95">".PLC"  COMPONENT SIDE SILKSCREEN</text>
-<text x="25.4" y="129.54" size="2.54" layer="95">".PLS"  SOLDER SIDE SILKSCREEN</text>
-<text x="25.4" y="124.46" size="2.54" layer="95">".CRC"  COMPONENT SIDE CREAM</text>
-<text x="25.4" y="119.38" size="2.54" layer="95">".CRS"  SOLDER SIDE CREAM</text>
+<text x="25.4" y="160.02" size="2.54" layer="95">".PLS"  SOLDER SIDE SILKSCREEN</text>
+<text x="25.4" y="154.94" size="2.54" layer="95">".CRC"  COMPONENT SIDE CREAM</text>
+<text x="25.4" y="149.86" size="2.54" layer="95">".CRS"  SOLDER SIDE CREAM</text>
 <text x="25.4" y="185.42" size="2.54" layer="95">".STC"  COMPONENT SIDE SOLDER MASK STOP</text>
-<text x="25.4" y="134.62" size="2.54" layer="95">".STS"  SOLDER SIDE SOLDER MASK STOP</text>
-<text x="25.4" y="109.22" size="2.54" layer="95">".DRD"  EXCELLON DRILL FILE</text>
-<text x="25.4" y="104.14" size="2.54" layer="95">".MNT"  XYRS DATA FILE FOR PLACEMENT</text>
+<text x="25.4" y="165.1" size="2.54" layer="95">".STS"  SOLDER SIDE SOLDER MASK STOP</text>
+<text x="25.4" y="139.7" size="2.54" layer="95">".DRD"  EXCELLON DRILL FILE</text>
+<text x="25.4" y="134.62" size="2.54" layer="95">".MNT"  XYRS DATA FILE FOR PLACEMENT</text>
 <text x="229.87" y="52.07" size="2.54" layer="95">LAYER 1 - COMPONENT SIDE, 1oz FINISH</text>
-<text x="229.87" y="46.99" size="2.54" layer="95">LAYER 2 - GROUND, 1/2oz</text>
-<text x="229.87" y="41.91" size="2.54" layer="95">LAYER 3 - INNER SIGNAL LAYER, 1/2oz</text>
-<text x="229.87" y="31.75" size="2.54" layer="95">LAYER 4 - GROUND , 1/2oz</text>
-<text x="229.87" y="26.67" size="2.54" layer="95">LAYER 5 - POWER, 1/2oz</text>
-<text x="229.87" y="16.51" size="2.54" layer="95">LAYER 6 - INNER SIGNAL LAYER, 1/2oz</text>
-<text x="229.87" y="11.43" size="2.54" layer="95">LAYER 7 - GROUND, 1/2oz</text>
-<text x="229.87" y="6.35" size="2.54" layer="95">LAYER 8 - SOLDER SIDE, 1oz FINISH</text>
+<text x="229.87" y="6.35" size="2.54" layer="95">LAYER 2 - SOLDER SIDE, 1oz FINISH</text>
 <text x="101.219" y="36.957" size="2.54" layer="95">DIELECTRIC THICKNESSES</text>
-<text x="181.61" y="49.53" size="2.1844" layer="95">6 mil</text>
-<text x="181.61" y="8.89" size="2.1844" layer="95">6 mil</text>
-<text x="181.61" y="44.45" size="2.1844" layer="95">6 mil</text>
-<text x="181.61" y="29.21" size="2.1844" layer="95">6 mil</text>
-<text x="181.61" y="13.97" size="2.1844" layer="95">6 mil</text>
-<text x="180.34" y="36.83" size="2.1844" layer="95">15 mil</text>
-<text x="180.34" y="21.59" size="2.1844" layer="95">15 mil</text>
+<text x="181.61" y="29.21" size="2.1844" layer="95">60 mil</text>
 <text x="161.417" y="63.119" size="3.175" layer="95">LAYER STACKUP DETAIL</text>
-<text x="16.51" y="97.79" size="2.54" layer="95">12. PLATED HOLE TOLERANCE  .003"</text>
-<text x="25.4" y="114.3" size="2.54" layer="97">".MIL"  MILLING LAYER FOR INNER CUTOUTS (NOT PLATED)</text>
+<text x="16.51" y="128.27" size="2.54" layer="95">12. PLATED HOLE TOLERANCE  .003"</text>
+<text x="25.4" y="144.78" size="2.54" layer="97">".MIL"  MILLING LAYER FOR INNER CUTOUTS (NOT PLATED)</text>
 <text x="17.78" y="203.2" size="2.54" layer="95">10. 15mil MAX RADIUS  INSIDE MILLING CORNERS FOR SMALL RECTANGULAR OPENINGS</text>
 <text x="25.4" y="175.26" size="2.54" layer="95">".DIM"  DIMENSION LAYER WITH OUTSIDE DIMENSIONS IN MM</text>
